Commit message: rover moves with wasd keys

File: rover/src/rover_description/urdf/rover.urdf (robot description, URDF)
Before this commit: robot differential_drive_rover, 6 links, 5 joints
Joints:
- joint front_left_wheel_joint: origin xyz=0.085 0.135 0 rpy=0 0 0 -> xyz=0.085 0.11 0 rpy=0 0 0
- joint front_right_wheel_joint: origin xyz=0.085 -0.135 0 rpy=0 0 0 -> xyz=0.085 -0.11 0 rpy=0 0 0
- joint rear_left_wheel_joint: origin xyz=-0.085 0.135 0 rpy=0 0 0 -> xyz=-0.085 0.11 0 rpy=0 0 0
- joint rear_right_wheel_joint: origin xyz=-0.085 -0.135 0 rpy=0 0 0 -> xyz=-0.085 -0.11 0 rpy=0 0 0

Commit message: Add simulated LiDAR and camera plugins

File: rover/src/rover_description/urdf/rover.urdf (robot description, URDF)
Before this commit: robot differential_drive_rover, 6 links, 5 joints
Links:
- added link camera_link, mass 0.05; collision box size=0.03 0.03 0.03; visual box size=0.03 0.03 0.03
- added link laser_link, mass 0.1; collision cylinder length=0.04 radius=0.05; visual cylinder length=0.04 radius=0.05
Joints:
- added joint camera_joint: type fixed, parent base_link, child camera_link, origin xyz=0.15 0 0.2 rpy=0 0 0
- added joint laser_joint: type fixed, parent base_link, child laser_link, origin xyz=0.1 0 0.1 rpy=0 0 0
